File: WT_Jlink_Adapter.kicad_pcb (KiCad board)
At the start: 2 copper layers, 12 x 27 mm, 4 parts, among them J1 Conn_02x10_Odd_Even, J2 Conn_02x05_Odd_Even

Commit message: Update Layout
Connections:
- net PIN7 renamed /PIN7
Other:
- board text added: "DBG"
- board text added: "GND"
- board text added: "RXD"
Changed lines of the file:
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@@
 	(net 11 "/SWCLK-TCK")
 	(net 12 "/VTREF")
-	(net 13 "PIN7")
+	(net 13 "/PIN7")
 	(footprint "Connector_PinSocket_2.54mm:PinSocket_2x10_P2.54mm_Horizontal"
 		(layer "F.Cu")
@@
 			(layers "*.Cu" "*.Mask")
 			(remove_unused_layers no)
-			(net 13 "PIN7")
+			(net 13 "/PIN7")
 			(pinfunction "C")
 			(pintype "passive")
@@
 			(layers "*.Cu" "*.Mask")
 			(remove_unused_layers no)
-			(net 13 "PIN7")
+			(net 13 "/PIN7")
 			(pinfunction "Pin_7")
 			(pintype "passive")
@@
 		(layer "Edge.Cuts")
 	)
+	(gr_text "GND"
+		(at 120.33 108.61 90)
+		(layer "F.SilkS")
+		(effects
+			(font
+				(size 1 1)
+				(thickness 0.1)
+			)
+			(justify left bottom)
+		)
+	)
+	(gr_text "DBG"
+		(at 120.33 111.61 90)
+		(layer "F.SilkS")
+		(effects
+			(font
+				(size 1 1)
+				(thickness 0.1)
+			)
+			(justify left bottom)
+		)
+	)
+	(gr_text "RXD"
+		(at 120.33 114.61 90)
+		(layer "F.SilkS")
+		(effects
+			(font
+				(size 1 1)
+				(thickness 0.1)
+			)
+			(justify left bottom)
+		)
+	)
 	(gr_text "1"
