File: WT_Jlink_Adapter.kicad_sch (KiCad schematic)
At the start: 4 parts, among them J1 Conn_02x10_Odd_Even, J2 Conn_02x05_Odd_Even

Commit message: Update Layout
Changed lines of the file:
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@@
 	(wire
 		(pts
-			(xy 144.78 91.44) (xy 139.7 91.44)
-		)
-		(stroke
-			(width 0)
-			(type default)
-		)
-	)
-	(wire
-		(pts
-			(xy 163.83 88.9) (xy 157.48 88.9)
+			(xy 157.48 88.9) (xy 168.91 88.9)
 		)
 		(stroke
@@
 	(wire
 		(pts
+			(xy 133.35 91.44) (xy 144.78 91.44)
+		)
+		(stroke
+			(width 0)
+			(type default)
+		)
+	)
+	(wire
+		(pts
 			(xy 93.98 95.25) (xy 82.55 95.25)
 		)
@@
 	(wire
 		(pts
-			(xy 157.48 91.44) (xy 163.83 91.44)
+			(xy 157.48 91.44) (xy 168.91 91.44)
 		)
 		(stroke
@@
 	(wire
 		(pts
-			(xy 157.48 93.98) (xy 163.83 93.98)
+			(xy 157.48 93.98) (xy 168.91 93.98)
 		)
 		(stroke
@@
 		)
 	)
+	(label "PIN7"
+		(at 133.35 91.44 0)
+		(fields_autoplaced yes)
+		(effects
+			(font
+				(size 1.27 1.27)
+			)
+			(justify left bottom)
+		)
+	)
 	(label "RXD"
 		(at 125.73 115.57 0)
@@
 		)
 	)
+	(label "PIN7"
+		(at 139.7 121.92 0)
+		(fields_autoplaced yes)
+		(effects
+			(font
+				(size 1.27 1.27)
+			)
+			(justify left bottom)
+		)
+	)
 	(label "SWO-TDO"
 		(at 82.55 95.25 0)
@@
 		)
 	)
-	(global_label "PIN7"
-		(shape input)
-		(at 139.7 91.44 180)
-		(effects
-			(font
-				(size 1.27 1.27)
-			)
-			(justify right)
-		)
-		(property "Intersheetrefs" "${INTERSHEET_REFS}"
-			(at 139.7 91.44 0)
-			(effects
-				(font
-					(size 1.27 1.27)
-				)
-				(hide yes)
-			)
-		)
-	)
-	(global_label "PIN7"
-		(shape input)
-		(at 139.7 121.92 0)
-		(effects
-			(font
-				(size 1.27 1.27)
-			)
-			(justify left)
-		)
-		(property "Intersheetrefs" "${INTERSHEET_REFS}"
-			(at 139.7 121.92 0)
-			(effects
-				(font
-					(size 1.27 1.27)
-				)
-				(hide yes)
-			)
-		)
-	)
